File: ElecExtern/ElecExtern.sch (KiCad schematic (older format))
At the start: 22 parts, among them J1 Conn_01x02, J2 Conn_01x04, J3 Conn_01x02, J4 Conn_01x02, J5 Conn_01x02, Q1 Q_NMOS_DGS, Q2 Q_NMOS_DGS, U1 R-78C3.3-1.0, U2 PMOS, U3 Xbee802.15.4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

Commit message: Grosse mise à jour
Parts:
- removed A1: Arduino_Nano_v3.x, Module:Arduino_Nano, symbol MCU_Module:Arduino_Nano_v3.x
- removed JP1: SolderJumper_2_Open, Resistor_SMD:R_1206_3216Metric_Pad1.42x1.75mm_HandSolder, symbol Jumper:SolderJumper_2_Open
- removed Q1, Q2: Q_NMOS_DGS, Package_TO_SOT_THT:TO-92L_Inline_Wide, symbol Device:Q_NMOS_DGS
- removed U1: R-78C3.3-1.0, Converter_DCDC:Converter_DCDC_RECOM_R-78E-0.5_THT, symbol Regulator_Switching:R-78C3.3-1.0
- added J6: Conn_01x02, Connector_PinHeader_2.54mm:PinHeader_1x02_P2.54mm_Vertical, symbol Connector_Generic:Conn_01x02
- added U1: AMS1117-3.3, Package_TO_SOT_SMD:SOT-223-3_TabPin2, symbol Regulator_Linear:AMS1117-3.3
- added U5: R-78C5.0-1.0, Converter_DCDC:Converter_DCDC_RECOM_R-78E-0.5_THT, symbol Regulator_Switching:R-78C5.0-1.0
- added U6: TEENSY3.2, RTS:TEENSY3.2_RTS, symbol PI06:TEENSY3.2
- C2: value C -> 10uF_tantalum_AMS1117; footprint Capacitor_SMD:C_1206_3216Metric_Pad1.42x1.75mm_HandSolder -> Capacitor_Tantalum_SMD:CP_EIA-3216-18_Kemet-A_Pad1.58x1.35mm_HandSolder
- C3: value 10uF -> 10uf MLCC; footprint Capacitor_SMD:C_1206_3216Metric_Pad1.42x1.75mm_HandSolder -> Capacitor_Tantalum_SMD:CP_EIA-3216-18_Kemet-A_Pad1.58x1.35mm_HandSolder
- R3, R4: value 1kR pull-up -> R
Connections:
- net RX_Duino is gone; now on net +3V3: R3.2
- net +12V: now also U1.3 (VI), U5.1 (IN); no longer C2.1
- net +3V3: now also C2.1, J2.2 (Pin_2), R4.2, U4.2 (VCC), U1.2 (VO); no longer C3.1, R4.1
- net +5V: now also C3.1, J6.1 (Pin_1), U5.3 (OUT), U6.28 (VIN(3.6-6.0V)); no longer J2.2 (Pin_2), R3.1, U4.2 (VCC)
- net Bouton1_IN: now also U6.8 (6(PWM))
- net Bouton2_IN: now also U6.9 (7(RX3))
- net DIN: now also U6.3 (1(TX1)); no longer R4.2
- net DOUT: now also U6.2 (0(RX1))
- net GND: now also J6.2 (Pin_2), U1.1 (GND), U5.2 (GND), U6.1 (GND), U6.27 (AGND), U6.31 (GND)
- net IO1: now also U6.5 (3(PWM))
- net IO2: now also U6.6 (4(PWM))
- net IO3: now also U6.7 (5(PWM))
- net MISO: now also U6.14 (12(MISO))
- net MOSI: now also U6.13 (11(MOSI))
- net PWM0_XBEE: now also U6.17 (15(A1))
- net PWM1_XBEE: now also U6.16 (14(A0))
- net SCK: now also U6.15 (13(SCK))
- net SCL: now also R4.1, U6.21 (19(A5/SCL0))
- net SDA: now also R3.1, U6.20 (18(A4/SDA0))
- net Xbee-reset: now also U6.4 (2)
- net ~CS: now also U6.12 (10(TX2/PWM))
- no-connect marks 22 -> 25
Other:
- note added: "Connexions UART\nTeensy <-> Xbee"
- note added: "Etage \nAlimentation\n"
- note added: "Interface I2C vers ecran LCD"
- note added: "LED power"
- note added: "Resistances pull-up I2C"
- note removed: "Arduino (5V) -> Xbee(3.3V)"
- note removed: "Arduino -> Ecran LCD par I2C\n"
- note removed: "Arduino: \nD13 = SCK\nD12 = MISO\nD11 = MOSI\nD10 = ~CS"
- note removed: "Mono-directionnal level shifters"
- note removed: "Note:\nL'ATmega328p a une tension\n d'entrée haute (Vih) égale à 0.6*Vcc\nPour Vcc = 5V, Vih = 3V.\n Le signal 3.3V de la Xbee est donc valide.\nEn théorie, pas besoin de level shifter 3.3V->5V"
- note removed: "On garde la possibilité\nd'en ajouter un, et on met un jumper soudé\n(Resistance 0Ohm) pour relier DOUT à RX Arduino"
- note removed: "REGULATEUR\nRECOM 3.3V"
- note removed: "Xbee (3.3V) -> Arduino (5V)"
- note removed: "Xbee fonctionne en 3.3V, Arduino en 5V.\n Pour eviter d'endommager le Xbee, on est obligés d'utiliser des level shifter."
- moved on the sheet: J2
